Commit message: Change robot colors

File: project2/my_robot/urdf/my_robot.xacro (robot description, xacro)
@@ -173,14 +173,14 @@
     </joint>
     <gazebo reference="left_wheel">
-        <material>Gazebo/Green</material>
+        <material>Gazebo/Blue</material>
     </gazebo>
     <gazebo reference="right_wheel">
-        <material>Gazebo/Green</material>
+        <material>Gazebo/Blue</material>
     </gazebo>
     <gazebo reference="chassis">
-        <material>Gazebo/Blue</material>
+        <material>Gazebo/Gold</material>
     </gazebo>
     <gazebo reference="camera">
-        <material>Gazebo/Red</material>
+        <material>Gazebo/Yellow</material>
     </gazebo>
 </robot>

Commit message: Change robot dimensions

File: project2/my_robot/urdf/my_robot.xacro (robot description, xacro)
@@ -22,5 +22,5 @@
             <origin xyz="0 0 0" rpy="0 0 0"/>
             <geometry>
-                <box size=".4 .2 .1"/>
+                <box size=".6 .4 .1"/>
             </geometry>
         </collision>
@@ -28,9 +28,9 @@
             <origin xyz="0 0 0" rpy="0 0 0"/>
             <geometry>
-                <box size=".4 .2 .1"/>
+                <box size=".6 .4 .1"/>
             </geometry>
         </visual>
         <collision name='back_caster_collision'>
-            <origin xyz="-0.15 0 -0.05" rpy="0 0 0"/>
+            <origin xyz="-0.25 0 -0.05" rpy="0 0 0"/>
             <geometry>
                 <sphere radius="0.0499"/>
@@ -38,5 +38,5 @@
         </collision>
         <visual name='back_caster_visual'>
-            <origin xyz="-0.15 0 -0.05" rpy="0 0 0"/>
+            <origin xyz="-0.25 0 -0.05" rpy="0 0 0"/>
             <geometry>
                 <sphere radius="0.05"/>
@@ -44,5 +44,5 @@
         </visual>
         <collision name='front_caster_collision'>
-            <origin xyz="0.15 0 -0.05" rpy="0 0 0"/>
+            <origin xyz="0.25 0 -0.05" rpy="0 0 0"/>
             <geometry>
                 <sphere radius="0.0499"/>
@@ -50,5 +50,5 @@
         </collision>
         <visual name='front_caster_visual'>
-            <origin xyz="0.15 0 -0.05" rpy="0 0 0"/>
+            <origin xyz="0.25 0 -0.05" rpy="0 0 0"/>
             <geometry>
                 <sphere radius="0.05"/>
@@ -139,5 +139,5 @@
     </link>
     <joint type="fixed" name="camera_joint">
-        <origin xyz="0.2 0 0" rpy="0 0 0"/>
+        <origin xyz="0.3 0 0" rpy="0 0 0"/>
         <axis xyz="0 1 0" rpy="0 0 0"/>
         <parent link="chassis"/>
@@ -167,5 +167,5 @@
     </link>
     <joint type="fixed" name="hokuyo_joint">
-        <origin xyz="0.15 0 0.1" rpy="0 0 0"/>
+        <origin xyz="0.25 0 0.1" rpy="0 0 0"/>
         <axis xyz="0 1 0" rpy="0 0 0"/>
         <parent link="chassis"/>
